File: Hardware/KiCad/antenna-test-board/antenna-test-board.kicad_pcb (KiCad board)
At the start: 2 copper layers, 50 x 80 mm, 5 parts, among them J1 50R

Commit message: refactor(kicad): una sola casa de bibliotecas, en v0-replica-sji/kicad-lib
Los modelos de la antena estaban en Hardware/KiCad/libraries/, que no es donde
esta registrada la biblioteca del proyecto. Resultado practico: al abrir KiCad
desde kicad-lib solo aparecia el LSM110A.

Se mueven a Hardware/v0-replica-sji/kicad-lib/, junto al LSM110A, en lugar de
duplicarlos. Duplicar bibliotecas KiCad es como se acaba editando el footprint
equivocado, y no hay forma de notar la deriva hasta que se fabrica.

Ahora la carpeta expone CINCO footprints bajo un unico nickname:

    0G-LockControl:LSM110A                              34 pads
    0G-LockControl:ANT_IFA_915MHz_LSM110A                2 pads (net tie)
    0G-LockControl:ANT_LSM110A_BreakAwaySlots_EVM_ONLY   0 pads
    0G-LockControl:C_0402_1005Metric_0G                  2 pads
    0G-LockControl:TP_Coax_50R_NanoVNA                   3 pads

mas dos bibliotecas de simbolos: 0G-LockControl (LSM110A) y 0G-Antenna.

Un solo path registrado en KiCad para todo el proyecto.

Comprobado antes de decidir el layout, no supuesto: el README anterior de
kicad-lib avisaba de que KiCad "espera" una carpeta .pretty y sugeria renombrar.
No hace falta. IO_MGR.PluginFind(KICAD_SEXP).FootprintEnumerate() enumera la
carpeta plana sin problema; el sufijo .pretty solo lo añade el dialogo de CREAR
biblioteca. Ese aviso se sustituye por el hecho verificado, con la advertencia
de NO renombrar la carpeta (la fp-lib-table y los campos Footprint apuntan a
este nombre).

Cambios de codigo:
  - antenna_geometry.py: nuevas constantes LIB_DIR, FP_LIB_NICKNAME,
    SYM_LIB_NICKNAME, SYM_LIB_FILE y helper lib_dir(). La ruta se define UNA vez
    porque son cuatro scripts los que tienen que coincidir; si se repitiera en
    cada uno, uno acabaria escribiendo donde otro no lee. lib_dir() resuelve
    contra la ubicacion del script y no contra el cwd, asi que los generadores
    dan el mismo resultado desde tools/, desde la raiz o desde CI.
  - gen_footprint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
Parts:
- ANT1: footprint 0G_Antenna:ANT_IFA_915MHz_LSM110A -> 0G-LockControl:ANT_IFA_915MHz_LSM110A
- C101, C102, L101: footprint 0G_RF:C_0402_1005Metric_0G -> 0G-LockControl:C_0402_1005Metric_0G
- J1: footprint 0G_RF:TP_Coax_50R_NanoVNA -> 0G-LockControl:TP_Coax_50R_NanoVNA
Changed lines of the file:
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@@
   (net 2 "ANT_FEED")
   (net 3 "RF_IN")
-  (footprint "0G_Antenna:ANT_IFA_915MHz_LSM110A" (layer "F.Cu")
+  (footprint "0G-LockControl:ANT_IFA_915MHz_LSM110A" (layer "F.Cu")
     (at 5.25 4)
     (descr "Antena IFA ranurada integrada en PCB para LSM110A. Banda 902-928 MHz (Sigfox RC2/RC4): el S11 medido por SJI da -16.4 dB a 902.1 MHz, -17.6 dB a 921.6 MHz y -29.3 dB a 928 MHz. NO sirve para EU868 sin reajustar: a 868.1 MHz el S11 de referencia es solo -8.7 dB (VSWR 2.17). Redibujo parametrico del plano '1.5 Antenna Dimension': placa 39.50 x 13.00 mm con dos ranuras de 0.50 mm que fuerzan un recorrido de corriente en forma de '2', stub en L de cortocircuito a GND y linea de alimentacion de 1.00 mm. Todo el cobre es un solo poligono. Origen del footprint = esquina superior izquierda del cobre. Requiere el borde superior de la PCB a 4.00 mm por encima del origen y el plano de tierra empezando exactamente a 16.03 mm por debajo. Footprint tipo net-tie: el pad 1 (FEED) y el pad 2 (GND) estan unidos a proposito por el stub, como en cualquier IFA.")
@@
     )
 )
-  (footprint "0G_RF:C_0402_1005Metric_0G" (layer "F.Cu")
+  (footprint "0G-LockControl:C_0402_1005Metric_0G" (layer "F.Cu")
     (at 38.415 23.3)
     (descr "Condensador 0402 (1005 metrico), land IPC nominal: 2 pads de 0.60 x 0.60 mm a +/-0.485 mm. Definido en el proyecto para no depender de las bibliotecas estandar de KiCad. Uso previsto: C101, condensador serie de acoplo/matching en la linea RF de la antena.")
@@
       (net 2 "ANT_FEED"))
 )
-  (footprint "0G_RF:C_0402_1005Metric_0G" (layer "F.Cu")
+  (footprint "0G-LockControl:C_0402_1005Metric_0G" (layer "F.Cu")
     (at 39.25 26.415 -90)
     (descr "Condensador 0402 (1005 metrico), land IPC nominal: 2 pads de 0.60 x 0.60 mm a +/-0.485 mm. Definido en el proyecto para no depender de las bibliotecas estandar de KiCad. Uso previsto: C101, condensador serie de acoplo/matching en la linea RF de la antena.")
@@
       (net 3 "RF_IN"))
 )
-  (footprint "0G_RF:C_0402_1005Metric_0G" (layer "F.Cu")
+  (footprint "0G-LockControl:C_0402_1005Metric_0G" (layer "F.Cu")
     (at 40.085 29.2 180)
     (descr "Condensador 0402 (1005 metrico), land IPC nominal: 2 pads de 0.60 x 0.60 mm a +/-0.485 mm. Definido en el proyecto para no depender de las bibliotecas estandar de KiCad. Uso previsto: C101, condensador serie de acoplo/matching en la linea RF de la antena.")
@@
       (net 3 "RF_IN"))
 )
-  (footprint "0G_RF:TP_Coax_50R_NanoVNA" (layer "F.Cu")
+  (footprint "0G-LockControl:TP_Coax_50R_NanoVNA" (layer "F.Cu")
     (at 39.25 34)
     (descr "Isla de 3 pads para soldar un pigtail coaxial de 50 ohm (RG-178 o semirrigido) y medir S11 con NanoVNA. Pad 1 = malla/GND izquierda, pad 2 = vivo, pad 3 = malla/GND derecha. La separacion vivo-malla es 0.15 mm, la misma del CPWG, para no crear discontinuidad. Solo para la placa de prueba y ajuste: no va en el producto.")
